File: schematics/kiCad/dds9851.sch (KiCad schematic (older format))
At the start: 28 parts, among them U1 901-144, U2 HC06, U3 901-144, U4 LTC6957HMS-4#PBF, U5 Teensy-LC, U6 MCP1700T-3302E_TT, U7 AD9851BRSZ, U8 901-144, U9 901-144

Commit message: pcb ready
Parts:
- removed U1, U3, U8, U9: 901-144, SMA_Female:SMA_Female, symbol SMA_Female:901-144
- added J1, J2, J3, J4: 2985-6004, 2985-6004:AMPHENOL_2985-6004, symbol 2985-6004:2985-6004
Connections:
- net GND: now also J1.S1, J1.S2, J1.S3, J1.S4, J2.S1, J2.S2, J2.S3, J2.S4, J3.S1, J3.S2, J3.S3, J3.S4, J4.S1, J4.S2, J4.S3, J4.S4
- net at U5.28 (21_A7_MOSI1_RX1): now also U7.8 (FQ__UD); no longer U7.22 (RESET)
- net at U5.29 (22_A8_SCL1_PWM_Touch): now also U7.22 (RESET); no longer U7.8 (FQ__UD)
- net at C1.2, R1.1: now also J1.1
- net at R4.2: now also J2.1
- net at R8.2, U7.20 (IOUTB): now also J4.1
- net at R7.1, U7.21 (IOUT): now also J3.1
Changed lines of the file:
@@
 Wire Wire Line
 	900  6400 1150 6400
-$Comp
-L SMA_Female:901-144 U1
-U 1 1 5F7F4767
-P 800 5850
-F 0 "U1" H 1532 5796 50  0000 L CNN
-F 1 "901-144" H 1532 5705 50  0000 L CNN
-F 2 "SMA_Female:SMA_Female" H 800 5850 50  0001 L BNN
-F 3 "901-144" H 800 5850 50  0001 L BNN
-F 4 "RF/COAXIAL, SMA JACK, STR, 50OHM, THD" H 800 5850 50  0001 L BNN "Field4"
-F 5 "98F1495" H 800 5850 50  0001 L BNN "Field5"
-F 6 "-" H 800 5850 50  0001 L BNN "Field6"
-F 7 "Amphenol" H 800 5850 50  0001 L BNN "Field7"
-	1    800  5850
-	0    -1   -1   0
-$EndComp
-Wire Wire Line
-	900  6350 900  6400
 Connection ~ 900  6400
-$Comp
-L SMA_Female:901-144 U3
-U 1 1 5F7FF45A
-P 2150 7600
-F 0 "U3" H 2882 7546 50  0000 L CNN
-F 1 "901-144" H 2882 7455 50  0000 L CNN
-F 2 "SMA_Female:SMA_Female" H 2150 7600 50  0001 L BNN
-F 3 "901-144" H 2150 7600 50  0001 L BNN
-F 4 "RF/COAXIAL, SMA JACK, STR, 50OHM, THD" H 2150 7600 50  0001 L BNN "Field4"
-F 5 "98F1495" H 2150 7600 50  0001 L BNN "Field5"
-F 6 "-" H 2150 7600 50  0001 L BNN "Field6"
-F 7 "Amphenol" H 2150 7600 50  0001 L BNN "Field7"
-	1    2150 7600
-	-1   0    0    1
-$EndComp
 $Comp
 L Device:R R4
 U 1 1 5F7FFE9C
 P 2900 7500
-F 0 "R4" H 2970 7546 50  0000 L CNN
-F 1 "450" H 2970 7455 50  0000 L CNN
+F 0 "R4" H 2700 7600 50  0000 L CNN
+F 1 "450" H 2700 7500 50  0000 L CNN
 F 2 "Resistor_SMD:R_1206_3216Metric_Pad1.42x1.75mm_HandSolder" V 2830 7500 50  0001 C CNN
 F 3 "~" H 2900 7500 50  0001 C CNN
@@
 Wire Wire Line
 	9400 1850 9400 1800
-$Comp
-L SMA_Female:901-144 U9
-U 1 1 5F846F9F
-P 9850 2750
-F 0 "U9" H 10582 2696 50  0000 L CNN
-F 1 "901-144" H 10582 2605 50  0000 L CNN
-F 2 "SMA_Female:SMA_Female" H 9850 2750 50  0001 L BNN
-F 3 "901-144" H 9850 2750 50  0001 L BNN
-F 4 "RF/COAXIAL, SMA JACK, STR, 50OHM, THD" H 9850 2750 50  0001 L BNN "Field4"
-F 5 "98F1495" H 9850 2750 50  0001 L BNN "Field5"
-F 6 "-" H 9850 2750 50  0001 L BNN "Field6"
-F 7 "Amphenol" H 9850 2750 50  0001 L BNN "Field7"
-	1    9850 2750
-	0    1    1    0
-$EndComp
-$Comp
-L SMA_Female:901-144 U8
-U 1 1 5F84948B
-P 9650 1650
-F 0 "U8" H 10382 1596 50  0000 L CNN
-F 1 "901-144" H 10382 1505 50  0000 L CNN
-F 2 "SMA_Female:SMA_Female" H 9650 1650 50  0001 L BNN
-F 3 "901-144" H 9650 1650 50  0001 L BNN
-F 4 "RF/COAXIAL, SMA JACK, STR, 50OHM, THD" H 9650 1650 50  0001 L BNN "Field4"
-F 5 "98F1495" H 9650 1650 50  0001 L BNN "Field5"
-F 6 "-" H 9650 1650 50  0001 L BNN "Field6"
-F 7 "Amphenol" H 9650 1650 50  0001 L BNN "Field7"
-	1    9650 1650
-	0    -1   -1   0
-$EndComp
 Wire Wire Line
 	9750 2150 9400 2150
 Connection ~ 9400 2150
-Wire Wire Line
-	9750 2250 9400 2250
-Connection ~ 9400 2250
 NoConn ~ 6950 3250
 $Comp
@@
 	4300 3150 4100 3150
 Wire Wire Line
-	6950 3550 4650 3550
-Wire Wire Line
-	4650 3550 4650 3250
-Wire Wire Line
 	4650 3250 4100 3250
-Wire Wire Line
-	6950 3650 4550 3650
-Wire Wire Line
-	4550 3650 4550 3350
-Wire Wire Line
-	4550 3350 4100 3350
-Wire Wire Line
-	6950 3750 4450 3750
-Wire Wire Line
-	4450 3750 4450 3450
 Wire Wire Line
 	4450 3450 4100 3450
@@
 	6950 1850 6950 1500
 $Comp
-L power:+3.3V #PWR?
+L power:+3.3V #PWR021
 U 1 1 5F8A6E89
 P 6800 2150
-F 0 "#PWR?" H 6800 2000 50  0001 C CNN
+F 0 "#PWR021" H 6800 2000 50  0001 C CNN
 F 1 "+3.3V" V 6800 2400 50  0000 C CNN
 F 2 "" H 6800 2150 50  0001 C CNN
@@
 	6800 2150 6950 2150
 Connection ~ 6950 2150
+Wire Wire Line
+	4650 3250 4650 3650
+Wire Wire Line
+	4650 3650 6950 3650
+Wire Wire Line
+	6950 3550 4750 3550
+Wire Wire Line
+	4750 3550 4750 3350
+Wire Wire Line
+	4100 3350 4750 3350
+Wire Wire Line
+	6950 3750 4450 3750
+Wire Wire Line
+	4450 3750 4450 3450
+$Comp
+L 2985-6004:2985-6004 J4
+U 1 1 5F885439
+P 9850 2350
+F 0 "J4" H 9690 2436 50  0000 R CNN
+F 1 "2985-6004" H 9690 2345 50  0000 R CNN
+F 2 "2985-6004:AMPHENOL_2985-6004" H 9850 2350 50  0001 L BNN
+F 3 "IPC-7351B" H 9850 2350 50  0001 L BNN
+F 4 "A" H 9850 2350 50  0001 L BNN "Field4"
+F 5 "9.79mm" H 9850 2350 50  0001 L BNN "Field5"
+F 6 "Amphenol" H 9850 2350 50  0001 L BNN "Field6"
+	1    9850 2350
+	-1   0    0    -1
+$EndComp
+Wire Wire Line
+	9750 2250 9400 2250
+Connection ~ 9400 2250
+Wire Wire Line
+	9750 2350 9750 2600
+Wire Wire Line
+	9750 2600 9400 2600
+Connection ~ 9400 2600
+$Comp
+L 2985-6004:2985-6004 J3
+U 1 1 5F898D06
+P 9850 2050
+F 0 "J3" H 9690 2044 50  0000 R CNN
+F 1 "2985-6004" H 9690 2135 50  0000 R CNN
+F 2 "2985-6004:AMPHENOL_2985-6004" H 9850 2050 50  0001 L BNN
+F 3 "IPC-7351B" H 9850 2050 50  0001 L BNN
+F 4 "A" H 9850 2050 50  0001 L BNN "Field4"
+F 5 "9.79mm" H 9850 2050 50  0001 L BNN "Field5"
+F 6 "Amphenol" H 9850 2050 50  0001 L BNN "Field6"
+	1    9850 2050
+	-1   0    0    1
+$EndComp
+Wire Wire Line
+	9750 2050 9750 1800
+Wire Wire Line
+	9750 1800 9400 1800
+Connection ~ 9400 1800
+$Comp
+L 2985-6004:2985-6004 J2
+U 1 1 5F8A6920
+P 2550 7600
+F 0 "J2" H 2542 7907 50  0000 C CNN
+F 1 "2985-6004" H 2542 7816 50  0000 C CNN
+F 2 "2985-6004:AMPHENOL_2985-6004" H 2550 7600 50  0001 L BNN
+F 3 "IPC-7351B" H 2550 7600 50  0001 L BNN
+F 4 "A" H 2550 7600 50  0001 L BNN "Field4"
+F 5 "9.79mm" H 2550 7600 50  0001 L BNN "Field5"
+F 6 "Amphenol" H 2550 7600 50  0001 L BNN "Field6"
+	1    2550 7600
+	1    0    0    -1
+$EndComp
+$Comp
+L power:GND #PWR019
+U 1 1 5F8AE060
+P 2800 7650
+F 0 "#PWR019" H 2800 7400 50  0001 C CNN
+F 1 "GND" H 2805 7477 50  0000 C CNN
+F 2 "" H 2800 7650 50  0001 C CNN
+F 3 "" H 2800 7650 50  0001 C CNN
+	1    2800 7650
+	0    -1   -1   0
+$EndComp
+Wire Wire Line
+	2800 7650 2650 7650
+Wire Wire Line
+	2650 7650 2650 7600
+$Comp
+L 2985-6004:2985-6004 J1
+U 1 1 5F8B276E
+P 800 6050
+F 0 "J1" V 746 6220 50  0000 L CNN
+F 1 "2985-6004" V 550 6100 50  0000 L CNN
+F 2 "2985-6004:AMPHENOL_2985-6004" H 800 6050 50  0001 L BNN
+F 3 "IPC-7351B" H 800 6050 50  0001 L BNN
+F 4 "A" H 800 6050 50  0001 L BNN "Field4"
+F 5 "9.79mm" H 800 6050 50  0001 L BNN "Field5"
+F 6 "Amphenol" H 800 6050 50  0001 L BNN "Field6"
+	1    800  6050
+	0    1    1    0
+$EndComp
+Wire Wire Line
+	900  6150 900  6400
+Wire Wire Line
+	800  6150 800  6950
+Wire Wire Line
+	800  6950 900  6950
+Connection ~ 900  6950
 $EndSCHEMATC
